Commit message: extracted robot dimensions into variables

File: ros2_ws/src/pepi_description/urdf/pepi.urdf.xacro (robot description, xacro)
@@ -1,4 +1,13 @@
 <?xml version="1.0"?>
-<robot name="pepi">
+<robot name="pepi" xmlns:xacro="http://www.ros.org/wiki/xacro">
+    <xacro:property name="base_lenght" value="0.325"/>
+    <xacro:property name="base_width" value="0.235"/>
+    <xacro:property name="base_thickness" value="0.018"/>
+    <xacro:property name="wheel_radius" value="0.0825"/>
+    <xacro:property name="wheel_thickness" value="0.045"/>
+    <xacro:property name="bottom_wheel_offset" value="0.015"/>
+    <xacro:property name="space_wheel_base" value="0.01"/>
+    <xacro:property name="caster_front_offset" value="0.08"/>
+    <xacro:property name="wheel_back_offset" value="0.095"/>
     <material name="body_color">
         <color rgba="0.5 0.5 0.5 1"/>
@@ -10,7 +19,7 @@
         <visual>
             <geometry>
-                <box size="0.35 0.235 0.018"/>
+                <box size="${base_lenght} ${base_width} ${base_thickness}"/>
             </geometry>
-            <origin xyz="0 0.0 0.009" rpy="0.0 0.0 0.0" />
+            <origin xyz="0 0.0 ${base_thickness/2}" rpy="0.0 0.0 0.0" />
             <material name="body_color"/>
         </visual>
@@ -19,7 +28,7 @@
         <visual>
             <geometry>
-                <cylinder radius="0.0825" length="0.045"/>
+                <cylinder radius="${wheel_radius}" length="${wheel_thickness}"/>
             </geometry>
-            <origin xyz="0.0 0.0 0.0" rpy="1.57 0.0 0.0"/>
+            <origin xyz="0.0 0.0 0.0" rpy="${pi/2.0} 0.0 0.0"/>
             <material name="wheel_color"/>
         </visual>
@@ -28,7 +37,7 @@
         <visual>
             <geometry>
-                <cylinder radius="0.0825" length="0.045"/>
+                <cylinder radius="${wheel_radius}" length="${wheel_thickness}"/>
             </geometry>
-            <origin xyz="0.0 0.0 0.0" rpy="1.57 0.0 0.0"/>
+            <origin xyz="0.0 0.0 0.0" rpy="${pi / 2.0} 0.0 0.0"/>
             <material name="wheel_color"/>
         </visual>
@@ -37,5 +46,5 @@
         <visual>
             <geometry>
-                <sphere radius="0.04875"/>
+                <sphere radius="${(bottom_wheel_offset + wheel_radius)/2}"/>
             </geometry>
             <origin xyz="0.0 0.0 0.0" rpy="0.0 0.0 0.0"/>
@@ -46,5 +55,5 @@
     </link>
     <joint name="base_right_wheel" type="continuous">
-        <origin xyz="-0.0675 -0.15 -0.015" rpy="0 0.0 0.0"/>
+        <origin xyz="-${base_lenght/2 - wheel_back_offset} -${base_width/2 + wheel_thickness/2 + bottom_wheel_offset} -${bottom_wheel_offset}" rpy="0 0.0 0.0"/>
         <parent link="base_link"/>
         <child link="right_wheel_link"/>
@@ -52,5 +61,5 @@
     </joint>
     <joint name="base_left_wheel" type="continuous">
-        <origin xyz="-0.0675 0.15 -0.015" rpy="0 0.0 0.0"/>
+        <origin xyz="-${base_lenght/2 - wheel_back_offset} ${base_width/2 + wheel_thickness/2 + bottom_wheel_offset} -${bottom_wheel_offset}" rpy="0 0.0 0.0"/>
         <parent link="base_link"/>
         <child link="left_wheel_link"/>
@@ -58,5 +67,5 @@
     </joint>
     <joint name="base_caster_wheel" type="fixed">
-        <origin xyz="0.0825 0.0 -0.04875" rpy="0.0 0.0 0.0"/>
+        <origin xyz="${base_lenght/2 - caster_front_offset} 0.0 -${(wheel_thickness/2 + bottom_wheel_offset)}" rpy="0.0 0.0 0.0"/>
         <parent link="base_link"/>
         <child link="caster_wheel_link"/>
@@ -64,5 +73,5 @@
     </joint>
     <joint name="base_foo" type="fixed">
-        <origin xyz="0.0 0.0 -0.0975"/>
+        <origin xyz="0.0 0.0 -${bottom_wheel_offset + wheel_radius}"/>
         <parent link="base_link"/>
         <child link="base_foot_link"/>

Commit message: splited pepi urdf file in common and mobile

File: ros2_ws/src/pepi_description/urdf/pepi.urdf.xacro (robot description, xacro)
@@ -1,80 +1,5 @@
 <?xml version="1.0"?>
 <robot name="pepi" xmlns:xacro="http://www.ros.org/wiki/xacro">
-    <xacro:property name="base_lenght" value="0.325"/>
-    <xacro:property name="base_width" value="0.235"/>
-    <xacro:property name="base_thickness" value="0.018"/>
-    <xacro:property name="wheel_radius" value="0.0825"/>
-    <xacro:property name="wheel_thickness" value="0.045"/>
-    <xacro:property name="bottom_wheel_offset" value="0.015"/>
-    <xacro:property name="space_wheel_base" value="0.01"/>
-    <xacro:property name="caster_front_offset" value="0.08"/>
-    <xacro:property name="wheel_back_offset" value="0.095"/>
-    <material name="body_color">
-        <color rgba="0.5 0.5 0.5 1"/>
-    </material>
-    <material name="wheel_color">
-        <color rgba="0.90 0.90 0.90 0.9"/>
-    </material>
-    <link name="base_link">
-        <visual>
-            <geometry>
-                <box size="${base_lenght} ${base_width} ${base_thickness}"/>
-            </geometry>
-            <origin xyz="0 0.0 ${base_thickness/2}" rpy="0.0 0.0 0.0" />
-            <material name="body_color"/>
-        </visual>
-    </link>
-    <link name="right_wheel_link">
-        <visual>
-            <geometry>
-                <cylinder radius="${wheel_radius}" length="${wheel_thickness}"/>
-            </geometry>
-            <origin xyz="0.0 0.0 0.0" rpy="${pi/2.0} 0.0 0.0"/>
-            <material name="wheel_color"/>
-        </visual>
-    </link>
-    <link name="left_wheel_link">
-        <visual>
-            <geometry>
-                <cylinder radius="${wheel_radius}" length="${wheel_thickness}"/>
-            </geometry>
-            <origin xyz="0.0 0.0 0.0" rpy="${pi / 2.0} 0.0 0.0"/>
-            <material name="wheel_color"/>
-        </visual>
-    </link>
-    <link name="caster_wheel_link">
-        <visual>
-            <geometry>
-                <sphere radius="${(bottom_wheel_offset + wheel_radius)/2}"/>
-            </geometry>
-            <origin xyz="0.0 0.0 0.0" rpy="0.0 0.0 0.0"/>
-            <material name="wheel_color"/>
-        </visual>
-    </link>
-    <link name="base_foot_link">
-    </link>
-    <joint name="base_right_wheel" type="continuous">
-        <origin xyz="-${base_lenght/2 - wheel_back_offset} -${base_width/2 + wheel_thickness/2 + bottom_wheel_offset} -${bottom_wheel_offset}" rpy="0 0.0 0.0"/>
-        <parent link="base_link"/>
-        <child link="right_wheel_link"/>
-        <axis xyz="0 1 0"/>
-    </joint>
-    <joint name="base_left_wheel" type="continuous">
-        <origin xyz="-${base_lenght/2 - wheel_back_offset} ${base_width/2 + wheel_thickness/2 + bottom_wheel_offset} -${bottom_wheel_offset}" rpy="0 0.0 0.0"/>
-        <parent link="base_link"/>
-        <child link="left_wheel_link"/>
-        <axis xyz="0 1 0"/>
-    </joint>
-    <joint name="base_caster_wheel" type="fixed">
-        <origin xyz="${base_lenght/2 - caster_front_offset} 0.0 -${(wheel_thickness/2 + bottom_wheel_offset)}" rpy="0.0 0.0 0.0"/>
-        <parent link="base_link"/>
-        <child link="caster_wheel_link"/>
-        <axis xyz="0.0 0.0 0.0"/>
-    </joint>
-    <joint name="base_foo" type="fixed">
-        <origin xyz="0.0 0.0 -${bottom_wheel_offset + wheel_radius}"/>
-        <parent link="base_link"/>
-        <child link="base_foot_link"/>
-        <axis xyz="0.0 0.0 0"/>
-    </joint>
+    <xacro:include filename="common_properties.xacro"/>
+    <xacro:include filename="mobile.xacro"/>
 </robot>
