Commit message: added collision

File: ros2_ws/src/pepi_description/urdf/common_properties.xacro (robot description, xacro)
@@ -7,3 +7,33 @@
         <color rgba="0.90 0.90 0.90 0.9"/>
     </material>
+    <xacro:macro name="box_inertia" params="m l w h xyz rpy">
+        <inertial>
+            <origin xyz="${xyz}" rpy="${rpy}"/>
+            <mass value="${m}"/>
+            <inertia
+                ixx="${(m/12) * (h*h + l*l)}" ixy="0.0" ixz="0.0"
+                iyy="${(m/12) * (w*w + l*l)}" iyz="0.0"
+                izz="${(m/12) * (w*w + h*h)}"/>
+        </inertial>
+    </xacro:macro>
+    <xacro:macro name="cylinder_inertia" params="m r w xyz rpy">
+        <inertial>
+            <origin xyz="${xyz}" rpy="${rpy}"/>
+            <mass value="${m}"/>
+            <inertia
+                ixx="${(m/12) * (3*r*r + w*w)}" ixy="0.0" ixz="0.0"
+                iyy="${(m/12) * (3*r*r + w*w)}" iyz="0.0"
+                izz="${(m/2) * r*r}"/>
+        </inertial>
+    </xacro:macro>
+    <xacro:macro name="sphere_inertia" params="m r xyz rpy">
+        <inertial>
+            <origin xyz="${xyz}" rpy="${rpy}"/>
+            <mass value="${m}"/>
+            <inertia
+                ixx="${(2/5) * m * r * r}" ixy="0.0" ixz="0.0"
+                iyy="${(2/5) * m * r * r}" iyz="0.0"
+                izz="${(2/5) * m * r * r}"/>
+        </inertial>
+    </xacro:macro>
 </robot>

File: ros2_ws/src/pepi_description/urdf/mobile.xacro (robot description, xacro)
@@ -18,4 +18,12 @@
             <material name="body_color"/>
         </visual>
+        <xacro:box_inertia m="5.0" l="${base_lenght}" w="${base_width}" h="${base_thickness}"
+            xyz="0 0.0 ${base_thickness/2}" rpy="0 0 0"/>
+        <collision>
+            <geometry>
+                <box size="${base_lenght} ${base_width} ${base_thickness}"/>
+            </geometry>
+            <origin xyz="0 0.0 ${base_thickness/2}" rpy="0.0 0.0 0.0" />
+        </collision>
     </link>
     <link name="right_wheel_link">
@@ -27,4 +35,12 @@
             <material name="wheel_color"/>
         </visual>
+        <xacro:cylinder_inertia m="1.5" r="${wheel_radius}" w="${wheel_thickness}"
+            xyz="0.0 0.0 0.0" rpy="${pi/2.0} 0.0 0.0"/>
+        <collision>
+            <geometry>
+                <cylinder radius="${wheel_radius}" length="${wheel_thickness}"/>
+            </geometry>
+            <origin xyz="0.0 0.0 0.0" rpy="${pi/2.0} 0.0 0.0"/>
+        </collision>
     </link>
     <link name="left_wheel_link">
@@ -36,4 +52,12 @@
             <material name="wheel_color"/>
         </visual>
+        <xacro:cylinder_inertia m="1.5" r="${wheel_radius}" w="${wheel_thickness}"
+            xyz="0.0 0.0 0.0" rpy="${pi/2.0} 0.0 0.0"/>
+        <collision>
+            <geometry>
+                <cylinder radius="${wheel_radius}" length="${wheel_thickness}"/>
+            </geometry>
+            <origin xyz="0.0 0.0 0.0" rpy="${pi / 2.0} 0.0 0.0"/>
+        </collision>
     </link>
     <link name="caster_wheel_link">
@@ -45,4 +69,12 @@
             <material name="wheel_color"/>
         </visual>
+        <xacro:sphere_inertia m="0.5" r="${(bottom_wheel_offset + wheel_radius)/2}"
+            xyz="0.0 0.0 0.0" rpy="0.0 0.0 0.0" />
+        <collision>
+            <geometry>
+                <sphere radius="${(bottom_wheel_offset + wheel_radius)/2}"/>
+            </geometry>
+            <origin xyz="0.0 0.0 0.0" rpy="0.0 0.0 0.0"/>
+        </collision>
     </link>
     <link name="base_foot_link">
